Commit message: feat: add real physics setup

File: urdf/left_leg.urdf.xacro (robot description, xacro)
@@ -92,5 +92,5 @@
       <dynamics damping="0.3" friction="0.04"/>
     </joint>
-    <gazebo reference="left_link7"><mu1>1.5</mu1><mu2>1.5</mu2><kp>1000000</kp><kd>10</kd></gazebo>
+    <gazebo reference="left_link7"><mu1>2.5</mu1><mu2>2.5</mu2><kp>1000000</kp><kd>10</kd></gazebo>
   </xacro:macro>
 </robot>

File: urdf/main.urdf.xacro (robot description, xacro)
@@ -4,4 +4,5 @@
   <xacro:arg name="controllers_file" default="$(find openleg_description)/config/controllers.yaml"/>
   <!-- Change these dimensions first when adapting the model to the real hardware. -->
+  <xacro:property name="base_mass" value="12.0"/>
   <xacro:property name="pelvis_x" value="0.18"/>
   <xacro:property name="pelvis_y" value="0.23358873"/>
@@ -32,8 +33,8 @@
     </collision>
     <inertial><origin xyz="0 0 ${pelvis_z / 2}" rpy="0 0 ${pi / 2}"/>
-      <mass value="8.0"/>
-      <inertia ixx="${8.0 * (pelvis_y**2 + pelvis_z**2) / 12}" ixy="0" ixz="0"
-               iyy="${8.0 * (pelvis_x**2 + pelvis_z**2) / 12}" iyz="0"
-               izz="${8.0 * (pelvis_x**2 + pelvis_y**2) / 12}"/>
+      <mass value="${base_mass}"/>
+      <inertia ixx="${base_mass * (pelvis_y**2 + pelvis_z**2) / 12}" ixy="0" ixz="0"
+               iyy="${base_mass * (pelvis_x**2 + pelvis_z**2) / 12}" iyz="0"
+               izz="${base_mass * (pelvis_x**2 + pelvis_y**2) / 12}"/>
     </inertial>
   </link>
@@ -57,5 +58,7 @@
   <xacro:if value="$(arg use_gazebo)">
     <ros2_control name="GazeboSimSystem" type="system">
-      <hardware><plugin>gz_ros2_control/GazeboSimSystem</plugin></hardware>
+      <hardware>
+        <plugin>gz_ros2_control/GazeboSimSystem</plugin>
+      </hardware>
       <xacro:position_controlled_joint joint_name="left_joint1"/>
       <xacro:position_controlled_joint joint_name="left_joint2"/>
@@ -71,14 +74,17 @@
       <xacro:position_controlled_joint joint_name="right_joint6"/>
     </ros2_control>
+    <!-- Simulated body IMU, mounted 70 mm above the base-link origin. -->
+    <gazebo reference="base_link">
+      <sensor name="base_imu" type="imu">
+        <pose>0 0 0.070 0 0 0</pose>
+        <always_on>true</always_on>
+        <update_rate>100</update_rate>
+        <topic>/imu</topic>
+      </sensor>
+    </gazebo>
     <gazebo>
       <plugin filename="libgz_ros2_control-system.so" name="gz_ros2_control::GazeboSimROS2ControlPlugin">
         <parameters>$(arg controllers_file)</parameters>
       </plugin>
-      <!-- Stable planar motion for the WASD + IK simulation controller. -->
-      <plugin filename="gz-sim-velocity-control-system" name="gz::sim::systems::VelocityControl"/>
-      <plugin filename="gz-sim-odometry-publisher-system" name="gz::sim::systems::OdometryPublisher">
-        <dimensions>3</dimensions>
-        <odom_publish_frequency>50</odom_publish_frequency>
-      </plugin>
     </gazebo>
   </xacro:if>

File: urdf/right_leg.urdf.xacro (robot description, xacro)
@@ -94,5 +94,5 @@
       <dynamics damping="0.3" friction="0.04"/>
     </joint>
-    <gazebo reference="right_link7"><mu1>1.5</mu1><mu2>1.5</mu2><kp>1000000</kp><kd>10</kd></gazebo>
+    <gazebo reference="right_link7"><mu1>2.5</mu1><mu2>2.5</mu2><kp>1000000</kp><kd>10</kd></gazebo>
   </xacro:macro>
 </robot>

Commit message: feat: add complete OpenLeg URDF and validated Gazebo walking demo

File: urdf/left_leg.urdf.xacro (robot description, xacro)
@@ -1,5 +1,5 @@
 <?xml version="1.0"?>
 <robot xmlns:xacro="http://www.ros.org/wiki/xacro">
-  <!-- One mesh origin drives both visual and collision geometry. -->
+  <!-- Non-foot visual and collision geometry share the same editable STL transform. -->
   <xacro:macro name="left_link_mesh" params="filename xyz rpy scale material">
     <visual>
@@ -14,5 +14,5 @@
   </xacro:macro>
   <!-- Mirrored six degree-of-freedom counterpart of the right leg. -->
-  <xacro:macro name="left_leg" params="parent hip_y link1_z upper_leg_length lower_leg_length foot_length foot_width foot_height">
+  <xacro:macro name="left_leg" params="parent hip_y link1_z upper_leg_length lower_leg_length foot_length foot_width foot_height foot_collision_width">
     <link name="left_link1">
       <xacro:left_link_mesh filename="package://openleg_description/meshes/left_leg/Left_Link1.stl" xyz="0 0 0" rpy="${pi / 2} 0 ${pi / 2}" scale="1 1 1" material="left_leg_blue"/>
@@ -30,6 +30,6 @@
       <parent link="left_link1"/><child link="left_link2"/>
       <origin xyz="0.064 0 0" rpy="0 ${pi} -${pi / 2}"/><axis xyz="0 -1 0"/>
-      <limit lower="-0.915" upper="${-0.915 + 5 * pi / 6}" effort="40" velocity="10.47198"/>
-      <dynamics damping="0.3" friction="0.05"/>
+      <limit lower="-0.915" upper="${-0.915 + 5 * pi / 6}" effort="140" velocity="10.47198"/>
+      <dynamics damping="2.0" friction="0.05"/>
     </joint>
     <link name="left_link3">
@@ -40,6 +40,6 @@
       <parent link="left_link2"/><child link="left_link3"/>
       <origin xyz="0.027 0.08001152 0" rpy="0 0 0"/><axis xyz="1 0 0"/>
-      <limit lower="-${pi / 6}" upper="${pi / 30}" effort="40" velocity="10.47198"/>
-      <dynamics damping="0.3" friction="0.05"/>
+      <limit lower="-${pi / 6}" upper="${pi / 9}" effort="140" velocity="10.47198"/>
+      <dynamics damping="2.0" friction="0.05"/>
     </joint>
     <link name="left_link4">
@@ -53,6 +53,6 @@
       <parent link="left_link3"/><child link="left_link4"/>
       <origin xyz="-0.027 0 0.074" rpy="0 0 0"/><axis xyz="0 0 -1"/>
-      <limit lower="-${pi / 2}" upper="${pi / 2}" effort="30" velocity="4.18879"/>
-      <dynamics damping="0.4" friction="0.05"/>
+      <limit lower="-${pi / 2}" upper="${pi / 2}" effort="97" velocity="4.18879"/>
+      <dynamics damping="2.5" friction="0.05"/>
     </joint>
     <link name="left_link5">
@@ -66,6 +66,6 @@
       <parent link="left_link4"/><child link="left_link5"/>
       <origin xyz="0 0.012 0.21175000"/><axis xyz="0 -1 0"/>
-      <limit lower="-${37 * pi / 72}" upper="${pi / 72}" effort="40" velocity="10.47198"/>
-      <dynamics damping="0.4" friction="0.05"/>
+      <limit lower="-${37 * pi / 72}" upper="${pi / 72}" effort="140" velocity="10.47198"/>
+      <dynamics damping="2.5" friction="0.05"/>
     </joint>
     <link name="left_link6">
@@ -76,9 +76,17 @@
       <parent link="left_link5"/><child link="left_link6"/>
       <origin xyz="0 -0.054 0.18"/><axis xyz="0 -1 0"/>
-      <limit lower="-${49 * pi / 360}" upper="${49 * pi / 360}" effort="40" velocity="10.47198"/>
-      <dynamics damping="0.3" friction="0.04"/>
+      <limit lower="-${49 * pi / 360}" upper="${49 * pi / 360}" effort="140" velocity="10.47198"/>
+      <dynamics damping="2.0" friction="0.04"/>
     </joint>
     <link name="left_link7">
-      <xacro:left_link_mesh filename="package://openleg_description/meshes/right_leg/Link7.stl" xyz="0 0 0" rpy="0 0 ${pi / 2}" scale="1 1 1" material="foot_black"/>
+      <visual>
+        <origin xyz="0 0 0" rpy="0 0 ${pi / 2}"/>
+        <geometry><mesh filename="package://openleg_description/meshes/right_leg/Link7.stl" scale="1 1 1"/></geometry>
+        <material name="foot_black"/>
+      </visual>
+      <collision>
+        <origin xyz="0.01 0 0.055"/>
+        <geometry><box size="${foot_length} ${foot_collision_width} ${foot_height}"/></geometry>
+      </collision>
       <inertial>
         <origin xyz="-0.025 0 -${foot_height / 2}"/><mass value="0.5"/>
@@ -89,8 +97,14 @@
       <parent link="left_link6"/><child link="left_link7"/>
       <origin xyz="-0.03712500 0.0385 0.12097726"/><axis xyz="1 0 0"/>
-      <limit lower="-${pi / 6}" upper="${pi / 6}" effort="30" velocity="4.18879"/>
-      <dynamics damping="0.3" friction="0.04"/>
+      <limit lower="-${pi / 6}" upper="${pi / 6}" effort="97" velocity="4.18879"/>
+      <dynamics damping="2.0" friction="0.04"/>
     </joint>
-    <gazebo reference="left_link7"><mu1>2.5</mu1><mu2>2.5</mu2><kp>1000000</kp><kd>10</kd></gazebo>
+    <gazebo reference="left_link1"><mu1>2.5</mu1><mu2>2.5</mu2><kp>200000</kp><kd>1000</kd><maxVel>0.05</maxVel><minDepth>0.001</minDepth></gazebo>
+    <gazebo reference="left_link2"><mu1>2.5</mu1><mu2>2.5</mu2><kp>200000</kp><kd>1000</kd><maxVel>0.05</maxVel><minDepth>0.001</minDepth></gazebo>
+    <gazebo reference="left_link3"><mu1>2.5</mu1><mu2>2.5</mu2><kp>200000</kp><kd>1000</kd><maxVel>0.05</maxVel><minDepth>0.001</minDepth></gazebo>
+    <gazebo reference="left_link4"><mu1>2.5</mu1><mu2>2.5</mu2><kp>200000</kp><kd>1000</kd><maxVel>0.05</maxVel><minDepth>0.001</minDepth></gazebo>
+    <gazebo reference="left_link5"><mu1>2.5</mu1><mu2>2.5</mu2><kp>200000</kp><kd>1000</kd><maxVel>0.05</maxVel><minDepth>0.001</minDepth></gazebo>
+    <gazebo reference="left_link6"><mu1>2.5</mu1><mu2>2.5</mu2><kp>200000</kp><kd>1000</kd><maxVel>0.05</maxVel><minDepth>0.001</minDepth></gazebo>
+    <gazebo reference="left_link7"><mu1>2.5</mu1><mu2>2.5</mu2><kp>200000</kp><kd>1000</kd><maxVel>0.05</maxVel><minDepth>0.001</minDepth></gazebo>
   </xacro:macro>
 </robot>

File: urdf/main.urdf.xacro (robot description, xacro)
@@ -4,15 +4,18 @@
   <xacro:arg name="controllers_file" default="$(find openleg_description)/config/controllers.yaml"/>
   <!-- Change these dimensions first when adapting the model to the real hardware. -->
-  <xacro:property name="base_mass" value="12.0"/>
+  <xacro:property name="base_mass" value="4.0"/>
   <xacro:property name="pelvis_x" value="0.18"/>
   <xacro:property name="pelvis_y" value="0.23358873"/>
   <xacro:property name="pelvis_z" value="0.26"/>
-  <xacro:property name="hip_spacing" value="0.060"/>
+  <!-- Inward test spacing: reduces the lateral COM transfer needed for one-leg support. -->
+  <xacro:property name="hip_spacing" value="0.000"/>
   <xacro:property name="link1_z" value="0.070"/>
   <xacro:property name="upper_leg_length" value="0.36"/>
   <xacro:property name="lower_leg_length" value="0.36"/>
-  <xacro:property name="foot_length" value="0.22"/>
-  <xacro:property name="foot_width" value="0.11"/>
-  <xacro:property name="foot_height" value="0.05"/>
+  <!-- Moderate single-support footprint: 200 x 140 x 30 mm. -->
+  <xacro:property name="foot_length" value="0.20"/>
+  <xacro:property name="foot_width" value="0.14"/>
+  <xacro:property name="foot_height" value="0.03"/>
+  <xacro:property name="foot_collision_width" value="0.14"/>
   <material name="pelvis_white"><color rgba="0.55 0.55 0.55 1"/></material>
   <material name="left_leg_blue"><color rgba="0.55 0.55 0.55 1"/></material>
@@ -41,8 +44,8 @@
   <xacro:left_leg parent="base_link" hip_y="${hip_spacing / 2}" link1_z="${link1_z}"
                   upper_leg_length="${upper_leg_length}" lower_leg_length="${lower_leg_length}"
-                  foot_length="${foot_length}" foot_width="${foot_width}" foot_height="${foot_height}"/>
+                  foot_length="${foot_length}" foot_width="${foot_width}" foot_height="${foot_height}" foot_collision_width="${foot_collision_width}"/>
   <xacro:right_leg parent="base_link" hip_y="-${hip_spacing / 2}" link1_z="${link1_z}"
                    upper_leg_length="${upper_leg_length}" lower_leg_length="${lower_leg_length}"
-                   foot_length="${foot_length}" foot_width="${foot_width}" foot_height="${foot_height}"/>
+                   foot_length="${foot_length}" foot_width="${foot_width}" foot_height="${foot_height}" foot_collision_width="${foot_collision_width}"/>
   <xacro:macro name="position_controlled_joint" params="joint_name">
     <joint name="${joint_name}">
@@ -76,4 +79,7 @@
     <!-- Simulated body IMU, mounted 70 mm above the base-link origin. -->
     <gazebo reference="base_link">
+      <mu1>2.5</mu1><mu2>2.5</mu2>
+      <kp>200000</kp><kd>1000</kd>
+      <maxVel>0.05</maxVel><minDepth>0.001</minDepth>
       <sensor name="base_imu" type="imu">
         <pose>0 0 0.070 0 0 0</pose>

File: urdf/right_leg.urdf.xacro (robot description, xacro)
@@ -1,5 +1,5 @@
 <?xml version="1.0"?>
 <robot xmlns:xacro="http://www.ros.org/wiki/xacro">
-  <!-- One editable origin drives both visual and collision for a mesh. -->
+  <!-- Non-foot visual and collision geometry share the same editable STL transform. -->
   <xacro:macro name="right_link_mesh" params="filename xyz rpy scale material">
     <visual>
@@ -14,5 +14,5 @@
   </xacro:macro>
   <!-- Right-side counterpart of the six degree-of-freedom left leg. -->
-  <xacro:macro name="right_leg" params="parent hip_y link1_z upper_leg_length lower_leg_length foot_length foot_width foot_height">
+  <xacro:macro name="right_leg" params="parent hip_y link1_z upper_leg_length lower_leg_length foot_length foot_width foot_height foot_collision_width">
     <!-- EDITABLE: Link 1 is the fixed leg mount; mesh xyz/rpy values are safe zeroed starting points. -->
     <link name="right_link1">
@@ -32,6 +32,6 @@
       <parent link="right_link1"/><child link="right_link2"/>
       <origin xyz="0.064 0 0" rpy="0 ${pi} -${pi / 2}"/><axis xyz="0 1 0"/>
-      <limit lower="-0.915" upper="${-0.915 + 5 * pi / 6}" effort="40" velocity="10.47198"/>
-      <dynamics damping="0.3" friction="0.05"/>
+      <limit lower="-0.915" upper="${-0.915 + 5 * pi / 6}" effort="140" velocity="10.47198"/>
+      <dynamics damping="2.0" friction="0.05"/>
     </joint>
     <link name="right_link3">
@@ -42,6 +42,6 @@
     <joint name="right_joint2" type="revolute">
       <parent link="right_link2"/><child link="right_link3"/><origin xyz="-0.027 0.08001152 0" rpy="0 0 0"/><axis xyz="1 0 0"/>
-      <limit lower="-${pi / 2}" upper="${pi / 6}" effort="40" velocity="10.47198"/>
-      <dynamics damping="0.3" friction="0.05"/>
+      <limit lower="-${pi / 2}" upper="${pi / 6}" effort="140" velocity="10.47198"/>
+      <dynamics damping="2.0" friction="0.05"/>
     </joint>
     <link name="right_link4">
@@ -55,6 +55,6 @@
     <joint name="right_joint3" type="revolute">
       <parent link="right_link3"/><child link="right_link4"/><origin xyz="0.027 0 0.074" rpy="0 0 0"/><axis xyz="0 0 1"/>
-      <limit lower="-${pi / 2}" upper="${pi / 2}" effort="30" velocity="4.18879"/>
-      <dynamics damping="0.4" friction="0.05"/>
+      <limit lower="-${pi / 2}" upper="${pi / 2}" effort="97" velocity="4.18879"/>
+      <dynamics damping="2.5" friction="0.05"/>
     </joint>
     <link name="right_link5">
@@ -68,6 +68,6 @@
     <joint name="right_joint4" type="revolute">
       <parent link="right_link4"/><child link="right_link5"/><origin xyz="0 0.012 0.21175000"/><axis xyz="0 1 0"/>
-      <limit lower="-${37 * pi / 72}" upper="${pi / 72}" effort="40" velocity="10.47198"/>
-      <dynamics damping="0.4" friction="0.05"/>
+      <limit lower="-${37 * pi / 72}" upper="${pi / 72}" effort="140" velocity="10.47198"/>
+      <dynamics damping="2.5" friction="0.05"/>
     </joint>
     <link name="right_link6">
@@ -78,9 +78,17 @@
     <joint name="right_joint5" type="revolute">
       <parent link="right_link5"/><child link="right_link6"/><origin xyz="0 -0.054 0.18"/><axis xyz="0 1 0"/>
-      <limit lower="-${49 * pi / 360}" upper="${49 * pi / 360}" effort="40" velocity="10.47198"/>
-      <dynamics damping="0.3" friction="0.04"/>
+      <limit lower="-${49 * pi / 360}" upper="${49 * pi / 360}" effort="140" velocity="10.47198"/>
+      <dynamics damping="2.0" friction="0.04"/>
     </joint>
     <link name="right_link7">
-      <xacro:right_link_mesh filename="package://openleg_description/meshes/right_leg/Link7.stl" xyz="0 0 0" rpy="0 0 -${pi / 2}" scale="1 1 1" material="foot_black"/>
+      <visual>
+        <origin xyz="0 0 0" rpy="0 0 -${pi / 2}"/>
+        <geometry><mesh filename="package://openleg_description/meshes/right_leg/Link7.stl" scale="1 1 1"/></geometry>
+        <material name="foot_black"/>
+      </visual>
+      <collision>
+        <origin xyz="-0.01 0 0.055"/>
+        <geometry><box size="${foot_length} ${foot_collision_width} ${foot_height}"/></geometry>
+      </collision>
       <inertial>
         <origin xyz="0.025 0 -${foot_height / 2}"/><mass value="0.5"/>
@@ -91,8 +99,14 @@
     <joint name="right_joint6" type="revolute">
       <parent link="right_link6"/><child link="right_link7"/><origin xyz="0.03712500 0.0385 0.12097726"/><axis xyz="1 0 0"/>
-      <limit lower="-${pi / 6}" upper="${pi / 6}" effort="30" velocity="4.18879"/>
-      <dynamics damping="0.3" friction="0.04"/>
+      <limit lower="-${pi / 6}" upper="${pi / 6}" effort="97" velocity="4.18879"/>
+      <dynamics damping="2.0" friction="0.04"/>
     </joint>
-    <gazebo reference="right_link7"><mu1>2.5</mu1><mu2>2.5</mu2><kp>1000000</kp><kd>10</kd></gazebo>
+    <gazebo reference="right_link1"><mu1>2.5</mu1><mu2>2.5</mu2><kp>200000</kp><kd>1000</kd><maxVel>0.05</maxVel><minDepth>0.001</minDepth></gazebo>
+    <gazebo reference="right_link2"><mu1>2.5</mu1><mu2>2.5</mu2><kp>200000</kp><kd>1000</kd><maxVel>0.05</maxVel><minDepth>0.001</minDepth></gazebo>
+    <gazebo reference="right_link3"><mu1>2.5</mu1><mu2>2.5</mu2><kp>200000</kp><kd>1000</kd><maxVel>0.05</maxVel><minDepth>0.001</minDepth></gazebo>
+    <gazebo reference="right_link4"><mu1>2.5</mu1><mu2>2.5</mu2><kp>200000</kp><kd>1000</kd><maxVel>0.05</maxVel><minDepth>0.001</minDepth></gazebo>
+    <gazebo reference="right_link5"><mu1>2.5</mu1><mu2>2.5</mu2><kp>200000</kp><kd>1000</kd><maxVel>0.05</maxVel><minDepth>0.001</minDepth></gazebo>
+    <gazebo reference="right_link6"><mu1>2.5</mu1><mu2>2.5</mu2><kp>200000</kp><kd>1000</kd><maxVel>0.05</maxVel><minDepth>0.001</minDepth></gazebo>
+    <gazebo reference="right_link7"><mu1>2.5</mu1><mu2>2.5</mu2><kp>200000</kp><kd>1000</kd><maxVel>0.05</maxVel><minDepth>0.001</minDepth></gazebo>
   </xacro:macro>
 </robot>
