Commit message: feat(sim): refine OpenLeg dynamics and body model
  - add waist and torso links with updated inertial properties
  - mirror leg dynamics and CAD-based mass properties
  - set DAMIAO torque limits and 24 V rated speed caps
  - tune foot, floor, and aluminium contact friction

File: urdf/left_leg.urdf.xacro (robot description, xacro)
@@ -1,14 +1,14 @@
 <?xml version="1.0"?>
 <robot xmlns:xacro="http://www.ros.org/wiki/xacro">
-  <!-- Non-foot visual and collision geometry share the same editable STL transform. -->
-  <xacro:macro name="left_link_mesh" params="filename xyz rpy scale material">
+  <!-- Non-foot visual and collision geometry use independent mesh files and share one editable transform. -->
+  <xacro:macro name="left_link_mesh" params="visual_filename collision_filename xyz rpy scale material">
     <visual>
       <origin xyz="${xyz}" rpy="${rpy}"/>
-      <geometry><mesh filename="${filename}" scale="${scale}"/></geometry>
+      <geometry><mesh filename="${visual_filename}" scale="${scale}"/></geometry>
       <material name="${material}"/>
     </visual>
     <collision>
       <origin xyz="${xyz}" rpy="${rpy}"/>
-      <geometry><mesh filename="${filename}" scale="${scale}"/></geometry>
+      <geometry><mesh filename="${collision_filename}" scale="${scale}"/></geometry>
     </collision>
   </xacro:macro>
@@ -16,6 +16,6 @@
   <xacro:macro name="left_leg" params="parent hip_y link1_z upper_leg_length lower_leg_length foot_length foot_width foot_height foot_collision_width">
     <link name="left_link1">
-      <xacro:left_link_mesh filename="package://openleg_description/meshes/left_leg/Left_Link1.stl" xyz="0 0 0" rpy="${pi / 2} 0 ${pi / 2}" scale="1 1 1" material="left_leg_blue"/>
-      <inertial><mass value="2.0"/><inertia ixx="0.00260" ixy="0" ixz="0" iyy="0.00260" iyz="0" izz="0.003025"/></inertial>
+      <xacro:left_link_mesh visual_filename="package://openleg_description/meshes/left_leg/Left_Link1.stl" collision_filename="package://openleg_description/meshes/left_leg/Left_Link1.stl" xyz="0 0 0" rpy="${pi / 2} 0 ${pi / 2}" scale="1 1 1" material="left_leg_blue"/>
+      <inertial><origin xyz="0.035 0 0"/><mass value="1.95"/><inertia ixx="0.003758080176" ixy="-0.000113110329" ixz="0.000018626355" iyy="0.002425144326" iyz="-0.000082610274" izz="0.002891882116"/></inertial>
     </link>
     <joint name="left_base_fixed_joint" type="fixed">
@@ -24,28 +24,28 @@
     </joint>
     <link name="left_link2">
-      <xacro:left_link_mesh filename="package://openleg_description/meshes/left_leg/Left_Link2.stl" xyz="0 0 0" rpy="0 ${pi} 0" scale="1 1 1" material="left_leg_blue"/>
-      <inertial><mass value="1.9"/><inertia ixx="0.00247" ixy="0" ixz="0" iyy="0.00247" iyz="0" izz="0.00287375"/></inertial>
+      <xacro:left_link_mesh visual_filename="package://openleg_description/meshes/left_leg/Left_Link2.stl" collision_filename="package://openleg_description/meshes/left_leg/Left_Link2.stl" xyz="0 0 0" rpy="0 ${pi} 0" scale="1 1 1" material="left_leg_blue"/>
+      <inertial><origin xyz="0 0.068 0"/><mass value="1.75"/><inertia ixx="0.003134759430" ixy="0.000015824529" ixz="0.000001019248" iyy="0.001856093868" iyz="-0.000000151933" izz="0.002351329675"/></inertial>
     </link>
     <joint name="left_joint1" type="revolute">
       <parent link="left_link1"/><child link="left_link2"/>
       <origin xyz="0.064 0 0" rpy="0 ${pi} -${pi / 2}"/><axis xyz="0 -1 0"/>
-      <limit lower="-0.915" upper="${-0.915 + 5 * pi / 6}" effort="140" velocity="10.47198"/>
+      <limit lower="-0.915" upper="${-0.915 + 5 * pi / 6}" effort="40" velocity="5.23599"/>
       <dynamics damping="2.0" friction="0.05"/>
     </joint>
     <link name="left_link3">
-      <xacro:left_link_mesh filename="package://openleg_description/meshes/right_leg/Link3.stl" xyz="0 0 0" rpy="0 0 -${pi / 2}" scale="1 1 1" material="joint_dark"/>
-      <inertial><origin xyz="-0.027 -0.08001152 0"/><mass value="0.3"/><inertia ixx="0.00039" ixy="0" ixz="0" iyy="0.00045375" iyz="0" izz="0.00039"/></inertial>
+      <xacro:left_link_mesh visual_filename="package://openleg_description/meshes/right_leg/Link3.stl" collision_filename="package://openleg_description/meshes/right_leg/Link3.stl" xyz="0 0 0" rpy="0 0 -${pi / 2}" scale="1 1 1" material="joint_dark"/>
+      <inertial><origin xyz="-0.001837 0 0.044592"/><mass value="0.25"/><inertia ixx="0.000271316138" ixy="0" ixz="0.000060712575" iyy="0.000291319338" iyz="0" izz="0.000136870384"/></inertial>
     </link>
     <joint name="left_joint2" type="revolute">
       <parent link="left_link2"/><child link="left_link3"/>
-      <origin xyz="0.027 0.08001152 0" rpy="0 0 0"/><axis xyz="1 0 0"/>
-      <limit lower="-${pi / 6}" upper="${pi / 9}" effort="140" velocity="10.47198"/>
+      <origin xyz="0.027 0.075 0" rpy="0 0 0"/><axis xyz="1 0 0"/>
+      <limit lower="-${pi / 2}" upper="${5 * pi / 36}" effort="40" velocity="5.23599"/>
       <dynamics damping="2.0" friction="0.05"/>
     </joint>
     <link name="left_link4">
-      <xacro:left_link_mesh filename="package://openleg_description/meshes/left_leg/Left_Link4.stl" xyz="0 0 0" rpy="-${pi / 2} 0 -${pi / 2}" scale="1 1 1" material="left_leg_blue"/>
+      <xacro:left_link_mesh visual_filename="package://openleg_description/meshes/left_leg/Left_Link4.stl" collision_filename="package://openleg_description/meshes/left_leg/Left_Link4.stl" xyz="0 0 0" rpy="-${pi / 2} 0 -${pi / 2}" scale="1 1 1" material="left_leg_blue"/>
       <inertial>
-        <origin xyz="0.027 0.074 -${upper_leg_length / 2}"/><mass value="2.75"/>
-        <inertia ixx="${2.75 * (0.09**2 + upper_leg_length**2) / 12}" ixy="0" ixz="0" iyy="${2.75 * (0.10**2 + upper_leg_length**2) / 12}" iyz="0" izz="${2.75 * (0.10**2 + 0.09**2) / 12}"/>
+        <origin xyz="0 -0.015 0.109"/><mass value="3.0"/>
+        <inertia ixx="0.011445270031" ixy="0.000000623481" ixz="0.000025390890" iyy="0.012149594340" iyz="0.001008737419" izz="0.003608626316"/>
       </inertial>
     </link>
@@ -53,28 +53,28 @@
       <parent link="left_link3"/><child link="left_link4"/>
       <origin xyz="-0.027 0 0.074" rpy="0 0 0"/><axis xyz="0 0 -1"/>
-      <limit lower="-${pi / 2}" upper="${pi / 2}" effort="97" velocity="4.18879"/>
+      <limit lower="-${pi / 2}" upper="${pi / 2}" effort="30" velocity="4.18879"/>
       <dynamics damping="2.5" friction="0.05"/>
     </joint>
     <link name="left_link5">
-      <xacro:left_link_mesh filename="package://openleg_description/meshes/left_leg/Left_Link5.stl" xyz="0 0 0" rpy="0 -${pi / 2} 0" scale="1 1 1" material="left_leg_blue"/>
+      <xacro:left_link_mesh visual_filename="package://openleg_description/meshes/right_leg/Link5.stl" collision_filename="package://openleg_description/meshes/right_leg/Link5.stl" xyz="0 0 0" rpy="0 -${pi / 2} 0" scale="1 1 1" material="left_leg_blue"/>
       <inertial>
-        <origin xyz="0 0 -${lower_leg_length / 2}"/><mass value="3.1"/>
-        <inertia ixx="${3.1 * (0.075**2 + lower_leg_length**2) / 12}" ixy="0" ixz="0" iyy="${3.1 * (0.09**2 + lower_leg_length**2) / 12}" iyz="0" izz="${3.1 * (0.09**2 + 0.075**2) / 12}"/>
+        <origin xyz="0 -0.014 0.129"/><mass value="1.94"/>
+        <inertia ixx="0.014234679170" ixy="0.000000064992" ixz="0.000000364381" iyy="0.013200580905" iyz="-0.000299782976" izz="0.002755133233"/>
       </inertial>
     </link>
     <joint name="left_joint4" type="revolute">
       <parent link="left_link4"/><child link="left_link5"/>
-      <origin xyz="0 0.012 0.21175000"/><axis xyz="0 -1 0"/>
-      <limit lower="-${37 * pi / 72}" upper="${pi / 72}" effort="140" velocity="10.47198"/>
+      <origin xyz="0 0.012 0.147"/><axis xyz="0 -1 0"/>
+      <limit lower="-${37 * pi / 72}" upper="${pi / 72}" effort="40" velocity="5.23599"/>
       <dynamics damping="2.5" friction="0.05"/>
     </joint>
     <link name="left_link6">
-      <xacro:left_link_mesh filename="package://openleg_description/meshes/left_leg/Left_Link6.stl" xyz="0 0 0" rpy="0 0 ${pi}" scale="1 1 1" material="joint_dark"/>
-      <inertial><mass value="1.0"/><inertia ixx="0.00060" ixy="0" ixz="0" iyy="0.00101667" iyz="0" izz="0.00060"/></inertial>
+      <xacro:left_link_mesh visual_filename="package://openleg_description/meshes/left_leg/Left_Link6.stl" collision_filename="package://openleg_description/meshes/left_leg/Left_Link6.stl" xyz="0 0 0" rpy="0 0 ${pi}" scale="1 1 1" material="joint_dark"/>
+      <inertial><origin xyz="0.004103 0.040339 0.077124"/><mass value="0.95"/><inertia ixx="0.000921950313" ixy="0.000031496560" ixz="-0.000005576139" iyy="0.000789173374" iyz="-0.000027795258" izz="0.000781461582"/></inertial>
     </link>
     <joint name="left_joint5" type="revolute">
       <parent link="left_link5"/><child link="left_link6"/>
-      <origin xyz="0 -0.054 0.18"/><axis xyz="0 -1 0"/>
-      <limit lower="-${49 * pi / 360}" upper="${49 * pi / 360}" effort="140" velocity="10.47198"/>
+      <origin xyz="0 -0.055 0.2"/><axis xyz="0 -1 0"/>
+      <limit lower="-${49 * pi / 360}" upper="${49 * pi / 360}" effort="30" velocity="4.18879"/>
       <dynamics damping="2.0" friction="0.04"/>
     </joint>
@@ -86,25 +86,25 @@
       </visual>
       <collision>
-        <origin xyz="0.01 0 0.055"/>
-        <geometry><box size="${foot_length} ${foot_collision_width} ${foot_height}"/></geometry>
+        <origin xyz="0 0 0" rpy="0 0 ${pi / 2}"/>
+        <geometry><mesh filename="package://openleg_description/meshes/right_leg/Link7.stl" scale="1 1 1"/></geometry>
       </collision>
       <inertial>
-        <origin xyz="-0.025 0 -${foot_height / 2}"/><mass value="0.5"/>
-        <inertia ixx="${0.5 * (foot_width**2 + foot_height**2) / 12}" ixy="0" ixz="0" iyy="${0.5 * (foot_length**2 + foot_height**2) / 12}" iyz="0" izz="${0.5 * (foot_length**2 + foot_width**2) / 12}"/>
+        <origin xyz="0.010 0 0.052"/><mass value="0.5"/>
+        <inertia ixx="0.000532780431" ixy="0" ixz="0.000013684277" iyy="0.001459897118" iyz="0" izz="0.001621743391"/>
       </inertial>
     </link>
     <joint name="left_joint6" type="revolute">
       <parent link="left_link6"/><child link="left_link7"/>
-      <origin xyz="-0.03712500 0.0385 0.12097726"/><axis xyz="1 0 0"/>
-      <limit lower="-${pi / 6}" upper="${pi / 6}" effort="97" velocity="4.18879"/>
+      <origin xyz="-0.032 0.043 0.08"/><axis xyz="1 0 0"/>
+      <limit lower="-${pi / 6}" upper="${pi / 6}" effort="30" velocity="4.18879"/>
       <dynamics damping="2.0" friction="0.04"/>
     </joint>
-    <gazebo reference="left_link1"><mu1>2.5</mu1><mu2>2.5</mu2><kp>200000</kp><kd>1000</kd><maxVel>0.05</maxVel><minDepth>0.001</minDepth></gazebo>
-    <gazebo reference="left_link2"><mu1>2.5</mu1><mu2>2.5</mu2><kp>200000</kp><kd>1000</kd><maxVel>0.05</maxVel><minDepth>0.001</minDepth></gazebo>
-    <gazebo reference="left_link3"><mu1>2.5</mu1><mu2>2.5</mu2><kp>200000</kp><kd>1000</kd><maxVel>0.05</maxVel><minDepth>0.001</minDepth></gazebo>
-    <gazebo reference="left_link4"><mu1>2.5</mu1><mu2>2.5</mu2><kp>200000</kp><kd>1000</kd><maxVel>0.05</maxVel><minDepth>0.001</minDepth></gazebo>
-    <gazebo reference="left_link5"><mu1>2.5</mu1><mu2>2.5</mu2><kp>200000</kp><kd>1000</kd><maxVel>0.05</maxVel><minDepth>0.001</minDepth></gazebo>
-    <gazebo reference="left_link6"><mu1>2.5</mu1><mu2>2.5</mu2><kp>200000</kp><kd>1000</kd><maxVel>0.05</maxVel><minDepth>0.001</minDepth></gazebo>
-    <gazebo reference="left_link7"><mu1>1.2</mu1><mu2>1.2</mu2><kp>200000</kp><kd>1000</kd><maxVel>0.05</maxVel><minDepth>0.001</minDepth></gazebo>
+    <gazebo reference="left_link1"><mu1>0.5</mu1><mu2>0.5</mu2><kp>200000</kp><kd>1000</kd><maxVel>0.05</maxVel><minDepth>0.001</minDepth></gazebo>
+    <gazebo reference="left_link2"><mu1>0.5</mu1><mu2>0.5</mu2><kp>200000</kp><kd>1000</kd><maxVel>0.05</maxVel><minDepth>0.001</minDepth></gazebo>
+    <gazebo reference="left_link3"><mu1>0.5</mu1><mu2>0.5</mu2><kp>200000</kp><kd>1000</kd><maxVel>0.05</maxVel><minDepth>0.001</minDepth></gazebo>
+    <gazebo reference="left_link4"><mu1>0.5</mu1><mu2>0.5</mu2><kp>200000</kp><kd>1000</kd><maxVel>0.05</maxVel><minDepth>0.001</minDepth></gazebo>
+    <gazebo reference="left_link5"><mu1>0.5</mu1><mu2>0.5</mu2><kp>200000</kp><kd>1000</kd><maxVel>0.05</maxVel><minDepth>0.001</minDepth></gazebo>
+    <gazebo reference="left_link6"><mu1>0.5</mu1><mu2>0.5</mu2><kp>200000</kp><kd>1000</kd><maxVel>0.05</maxVel><minDepth>0.001</minDepth></gazebo>
+    <gazebo reference="left_link7"><mu1>0.9</mu1><mu2>0.9</mu2><kp>200000</kp><kd>1000</kd><maxVel>0.05</maxVel><minDepth>0.001</minDepth></gazebo>
   </xacro:macro>
 </robot>

File: urdf/main.urdf.xacro (robot description, xacro)
@@ -4,5 +4,9 @@
   <xacro:arg name="controllers_file" default="$(find openleg_description)/config/controllers.yaml"/>
   <!-- Change these dimensions first when adapting the model to the real hardware. -->
-  <xacro:property name="base_mass" value="4.0"/>
+  <xacro:property name="base_mass" value="2.5"/>
+  <!-- EDITABLE: replace with the measured upper-body inertial data. -->
+  <xacro:property name="upper_body_mass" value="3.4"/>
+  <!-- EDITABLE: replace with the measured torso inertial data. -->
+  <xacro:property name="torso_mass" value="5.5"/>
   <xacro:property name="pelvis_x" value="0.18"/>
   <xacro:property name="pelvis_y" value="0.23358873"/>
@@ -10,5 +14,5 @@
   <!-- Inward test spacing: reduces the lateral COM transfer needed for one-leg support. -->
   <xacro:property name="hip_spacing" value="0.000"/>
-  <xacro:property name="link1_z" value="0.070"/>
+  <xacro:property name="link1_z" value="0.078"/>
   <xacro:property name="upper_leg_length" value="0.36"/>
   <xacro:property name="lower_leg_length" value="0.36"/>
@@ -35,11 +39,61 @@
       <geometry><mesh filename="package://openleg_description/meshes/base/Base.stl" scale="1 1 1"/></geometry>
     </collision>
-    <inertial><origin xyz="0 0 ${pelvis_z / 2}" rpy="0 0 ${pi / 2}"/>
+    <!-- Fusion inertia at COM, transformed into base_link axes and scaled for the 2.5 kg total mass. -->
+    <inertial><origin xyz="0.000013 0.000550 0.143563"/>
       <mass value="${base_mass}"/>
-      <inertia ixx="${base_mass * (pelvis_y**2 + pelvis_z**2) / 12}" ixy="0" ixz="0"
-               iyy="${base_mass * (pelvis_x**2 + pelvis_z**2) / 12}" iyz="0"
-               izz="${base_mass * (pelvis_x**2 + pelvis_y**2) / 12}"/>
+      <inertia ixx="0.010284366864" ixy="-0.000000073216" ixz="-0.000000349169"
+               iyy="0.012990553920" iyz="-0.000007596132" izz="0.007354536828"/>
     </inertial>
   </link>
+  <!-- Waist yaw: the UpperBody CAD origin is 207 mm above the base-link origin. -->
+  <link name="upper_body_link">
+    <visual>
+      <origin xyz="0 0 0" rpy="0 0 ${pi / 2}"/>
+      <geometry><mesh filename="package://openleg_description/meshes/base/UpperBody.stl" scale="1 1 1"/></geometry>
+      <material name="pelvis_white"/>
+    </visual>
+    <collision>
+      <origin xyz="0 0 0" rpy="0 0 ${pi / 2}"/>
+      <geometry><mesh filename="package://openleg_description/meshes/base/UpperBody.stl" scale="1 1 1"/></geometry>
+    </collision>
+    <!-- Fusion inertia at COM, transformed into upper_body_link axes and scaled for the 3.4 kg total mass. -->
+    <inertial>
+      <origin xyz="0.000019 0 0.067755"/>
+      <mass value="${upper_body_mass}"/>
+      <inertia ixx="0.009092410126" ixy="0" ixz="-0.000000147058" iyy="0.006325647511" iyz="-0.000000766627" izz="0.008640210279"/>
+    </inertial>
+  </link>
+  <joint name="waist_joint" type="revolute">
+    <parent link="base_link"/><child link="upper_body_link"/>
+    <origin xyz="0 0 0.207" rpy="0 0 0"/>
+    <axis xyz="0 0 1"/>
+    <limit lower="-${pi / 2}" upper="${pi / 2}" effort="40" velocity="5.23599"/>
+    <dynamics damping="2.0" friction="0.05"/>
+  </joint>
+  <!-- Torso pitch: the Torso CAD origin is 70 mm above the upper-body origin. -->
+  <link name="torso_link">
+    <visual>
+      <origin xyz="0 0 0" rpy="0 0 ${pi / 2}"/>
+      <geometry><mesh filename="package://openleg_description/meshes/base/Torso.stl" scale="1 1 1"/></geometry>
+      <material name="pelvis_white"/>
+    </visual>
+    <collision>
+      <origin xyz="0 0 0" rpy="0 0 ${pi / 2}"/>
+      <geometry><mesh filename="package://openleg_description/meshes/base/Torso.stl" scale="1 1 1"/></geometry>
+    </collision>
+    <!-- Provisional electronics and structure estimate; replace with Fusion values when the assembly is complete. -->
+    <inertial>
+      <origin xyz="0 0.065 0.110"/>
+      <mass value="${torso_mass}"/>
+      <inertia ixx="0.065980" ixy="0" ixz="0" iyy="0.060544" iyz="0" izz="0.034990"/>
+    </inertial>
+  </link>
+  <joint name="torso_pitch_joint" type="revolute">
+    <parent link="upper_body_link"/><child link="torso_link"/>
+    <origin xyz="0 -0.065 0.07" rpy="0 0 0"/>
+    <axis xyz="0 1 0"/>
+    <limit lower="-${pi / 6}" upper="${pi / 2}" effort="80" velocity="5.23599"/>
+    <dynamics damping="2.0" friction="0.05"/>
+  </joint>
   <xacro:left_leg parent="base_link" hip_y="${hip_spacing / 2}" link1_z="${link1_z}"
                   upper_leg_length="${upper_leg_length}" lower_leg_length="${lower_leg_length}"
@@ -76,8 +130,10 @@
       <xacro:position_controlled_joint joint_name="right_joint5"/>
       <xacro:position_controlled_joint joint_name="right_joint6"/>
+      <xacro:position_controlled_joint joint_name="waist_joint"/>
+      <xacro:position_controlled_joint joint_name="torso_pitch_joint"/>
     </ros2_control>
     <!-- Simulated body IMU, mounted 70 mm above the base-link origin. -->
     <gazebo reference="base_link">
-      <mu1>2.5</mu1><mu2>2.5</mu2>
+      <mu1>0.5</mu1><mu2>0.5</mu2>
       <kp>200000</kp><kd>1000</kd>
       <maxVel>0.05</maxVel><minDepth>0.001</minDepth>
@@ -89,4 +145,12 @@
       </sensor>
     </gazebo>
+    <gazebo reference="upper_body_link">
+      <mu1>0.5</mu1><mu2>0.5</mu2>
+      <kp>200000</kp><kd>1000</kd><maxVel>0.05</maxVel><minDepth>0.001</minDepth>
+    </gazebo>
+    <gazebo reference="torso_link">
+      <mu1>0.5</mu1><mu2>0.5</mu2>
+      <kp>200000</kp><kd>1000</kd><maxVel>0.05</maxVel><minDepth>0.001</minDepth>
+    </gazebo>
     <gazebo>
       <plugin filename="libgz_ros2_control-system.so" name="gz_ros2_control::GazeboSimROS2ControlPlugin">
