Commit message: feat(sim): refine OpenLeg dynamics and body model
  - add waist and torso links with updated inertial properties
  - mirror leg dynamics and CAD-based mass properties
  - set DAMIAO torque limits and 24 V rated speed caps
  - tune foot, floor, and aluminium contact friction

File: urdf/right_leg.urdf.xacro (robot description, xacro)
@@ -1,14 +1,14 @@
 <?xml version="1.0"?>
 <robot xmlns:xacro="http://www.ros.org/wiki/xacro">
-  <!-- Non-foot visual and collision geometry share the same editable STL transform. -->
-  <xacro:macro name="right_link_mesh" params="filename xyz rpy scale material">
+  <!-- Non-foot visual and collision geometry use independent mesh files and share one editable transform. -->
+  <xacro:macro name="right_link_mesh" params="visual_filename collision_filename xyz rpy scale material">
     <visual>
       <origin xyz="${xyz}" rpy="${rpy}"/>
-      <geometry><mesh filename="${filename}" scale="${scale}"/></geometry>
+      <geometry><mesh filename="${visual_filename}" scale="${scale}"/></geometry>
       <material name="${material}"/>
     </visual>
     <collision>
       <origin xyz="${xyz}" rpy="${rpy}"/>
-      <geometry><mesh filename="${filename}" scale="${scale}"/></geometry>
+      <geometry><mesh filename="${collision_filename}" scale="${scale}"/></geometry>
     </collision>
   </xacro:macro>
@@ -17,6 +17,7 @@
     <!-- EDITABLE: Link 1 is the fixed leg mount; mesh xyz/rpy values are safe zeroed starting points. -->
     <link name="right_link1">
-      <xacro:right_link_mesh filename="package://openleg_description/meshes/right_leg/Right_Link1.stl" xyz="0 0 0" rpy="${pi / 2} 0 ${pi / 2}" scale="1 1 1" material="right_leg_red"/>
-      <inertial><mass value="2.0"/><inertia ixx="0.00260" ixy="0" ixz="0" iyy="0.00260" iyz="0" izz="0.003025"/></inertial>
+      <xacro:right_link_mesh visual_filename="package://openleg_description/meshes/right_leg/Right_Link1.stl" collision_filename="package://openleg_description/meshes/right_leg/Right_Link1.stl" xyz="0 0 0" rpy="${pi / 2} 0 ${pi / 2}" scale="1 1 1" material="right_leg_red"/>
+      <!-- Fusion inertia at COM, transformed into this URDF frame and scaled for the 1.95 kg total link mass. -->
+      <inertial><origin xyz="0.035 0 0"/><mass value="1.95"/><inertia ixx="0.003758080176" ixy="0.000113110329" ixz="0.000018626355" iyy="0.002425144326" iyz="0.000082610274" izz="0.002891882116"/></inertial>
     </link>
     <joint name="right_base_fixed_joint" type="fixed">
@@ -25,6 +26,6 @@
     </joint>
     <link name="right_link2">
-      <xacro:right_link_mesh filename="package://openleg_description/meshes/right_leg/Right_Link2.stl" xyz="0 0 0" rpy="0 0 0" scale="1 1 1" material="right_leg_red"/>
-      <inertial><mass value="1.9"/><inertia ixx="0.00247" ixy="0" ixz="0" iyy="0.00247" iyz="0" izz="0.00287375"/></inertial>
+      <xacro:right_link_mesh visual_filename="package://openleg_description/meshes/right_leg/Right_Link2.stl" collision_filename="package://openleg_description/meshes/right_leg/Right_Link2.stl" xyz="0 0 0" rpy="0 0 0" scale="1 1 1" material="right_leg_red"/>
+      <inertial><origin xyz="0 0.068 0"/><mass value="1.75"/><inertia ixx="0.003134759430" ixy="-0.000015824529" ixz="-0.000001019248" iyy="0.001856093868" iyz="-0.000000151933" izz="0.002351329675"/></inertial>
     </link>
     <!-- J1: hip pitch, Link1 -> Link2 -->
@@ -32,22 +33,22 @@
       <parent link="right_link1"/><child link="right_link2"/>
       <origin xyz="0.064 0 0" rpy="0 ${pi} -${pi / 2}"/><axis xyz="0 1 0"/>
-      <limit lower="-0.915" upper="${-0.915 + 5 * pi / 6}" effort="140" velocity="10.47198"/>
+      <limit lower="-0.915" upper="${-0.915 + 5 * pi / 6}" effort="40" velocity="5.23599"/>
       <dynamics damping="2.0" friction="0.05"/>
     </joint>
     <link name="right_link3">
-      <xacro:right_link_mesh filename="package://openleg_description/meshes/right_leg/Link3.stl" xyz="0 0 0" rpy="0 0 ${pi / 2}" scale="1 1 1" material="joint_dark"/>
-      <inertial><origin xyz="0.027 -0.08001152 0"/><mass value="0.3"/><inertia ixx="0.00039" ixy="0" ixz="0" iyy="0.00045375" iyz="0" izz="0.00039"/></inertial>
+      <xacro:right_link_mesh visual_filename="package://openleg_description/meshes/right_leg/Link3.stl" collision_filename="package://openleg_description/meshes/right_leg/Link3.stl" xyz="0 0 0" rpy="0 0 ${pi / 2}" scale="1 1 1" material="joint_dark"/>
+      <inertial><origin xyz="0.001837 0 0.044592"/><mass value="0.25"/><inertia ixx="0.000271316138" ixy="0" ixz="-0.000060712575" iyy="0.000291319338" iyz="0" izz="0.000136870384"/></inertial>
     </link>
     <!-- J2: hip roll, Link2 -> Link3 -->
     <joint name="right_joint2" type="revolute">
-      <parent link="right_link2"/><child link="right_link3"/><origin xyz="-0.027 0.08001152 0" rpy="0 0 0"/><axis xyz="1 0 0"/>
-      <limit lower="-${pi / 2}" upper="${pi / 6}" effort="140" velocity="10.47198"/>
+      <parent link="right_link2"/><child link="right_link3"/><origin xyz="-0.027 0.075 0" rpy="0 0 0"/><axis xyz="1 0 0"/>
+      <limit lower="-${pi / 2}" upper="${5 * pi / 36}" effort="40" velocity="5.23599"/>
       <dynamics damping="2.0" friction="0.05"/>
     </joint>
     <link name="right_link4">
-      <xacro:right_link_mesh filename="package://openleg_description/meshes/right_leg/Right_Link4.stl" xyz="0 0 0" rpy="-${pi / 2} 0 -${pi / 2}" scale="1 1 1" material="right_leg_red"/>
+      <xacro:right_link_mesh visual_filename="package://openleg_description/meshes/right_leg/Right_Link4.stl" collision_filename="package://openleg_description/meshes/right_leg/Right_Link4.stl" xyz="0 0 0" rpy="-${pi / 2} 0 -${pi / 2}" scale="1 1 1" material="right_leg_red"/>
       <inertial>
-        <origin xyz="-0.027 0.074 -${upper_leg_length / 2}"/><mass value="2.75"/>
-        <inertia ixx="${2.75 * (0.09**2 + upper_leg_length**2) / 12}" ixy="0" ixz="0" iyy="${2.75 * (0.10**2 + upper_leg_length**2) / 12}" iyz="0" izz="${2.75 * (0.10**2 + 0.09**2) / 12}"/>
+        <origin xyz="0 -0.015 0.109"/><mass value="3.0"/>
+        <inertia ixx="0.011445270031" ixy="-0.000000623481" ixz="-0.000025390890" iyy="0.012149594340" iyz="0.001008737419" izz="0.003608626316"/>
       </inertial>
     </link>
@@ -55,28 +56,29 @@
     <joint name="right_joint3" type="revolute">
       <parent link="right_link3"/><child link="right_link4"/><origin xyz="0.027 0 0.074" rpy="0 0 0"/><axis xyz="0 0 1"/>
-      <limit lower="-${pi / 2}" upper="${pi / 2}" effort="97" velocity="4.18879"/>
+      <limit lower="-${pi / 2}" upper="${pi / 2}" effort="30" velocity="4.18879"/>
       <dynamics damping="2.5" friction="0.05"/>
     </joint>
     <link name="right_link5">
-      <xacro:right_link_mesh filename="package://openleg_description/meshes/right_leg/Right_Link5.stl" xyz="0 0 0" rpy="0 -${pi / 2} 0" scale="1 1 1" material="right_leg_red"/>
+      <xacro:right_link_mesh visual_filename="package://openleg_description/meshes/right_leg/Link5.stl" collision_filename="package://openleg_description/meshes/right_leg/Link5.stl" xyz="0 0 0" rpy="0 -${pi / 2} 0" scale="1 1 1" material="right_leg_red"/>
       <inertial>
-        <origin xyz="0 0 -${lower_leg_length / 2}"/><mass value="3.1"/>
-        <inertia ixx="${3.1 * (0.075**2 + lower_leg_length**2) / 12}" ixy="0" ixz="0" iyy="${3.1 * (0.09**2 + lower_leg_length**2) / 12}" iyz="0" izz="${3.1 * (0.09**2 + 0.075**2) / 12}"/>
+        <origin xyz="0 -0.014 0.129"/><mass value="1.94"/>
+        <inertia ixx="0.014234679170" ixy="-0.000000064992" ixz="-0.000000364381" iyy="0.013200580905" iyz="-0.000299782976" izz="0.002755133233"/>
       </inertial>
     </link>
     <!-- J4: knee pitch, Link4 -> Link5 -->
     <joint name="right_joint4" type="revolute">
-      <parent link="right_link4"/><child link="right_link5"/><origin xyz="0 0.012 0.21175000"/><axis xyz="0 1 0"/>
-      <limit lower="-${37 * pi / 72}" upper="${pi / 72}" effort="140" velocity="10.47198"/>
+      <parent link="right_link4"/><child link="right_link5"/><origin xyz="0 0.012 0.147"/><axis xyz="0 1 0"/>
+      <limit lower="-${37 * pi / 72}" upper="${pi / 72}" effort="40" velocity="5.23599"/>
       <dynamics damping="2.5" friction="0.05"/>
     </joint>
     <link name="right_link6">
-      <xacro:right_link_mesh filename="package://openleg_description/meshes/right_leg/Right_Link6.stl" xyz="0 0 0" rpy="0 0 ${pi}" scale="1 1 1" material="joint_dark"/>
-      <inertial><mass value="1.0"/><inertia ixx="0.00060" ixy="0" ixz="0" iyy="0.00101667" iyz="0" izz="0.00060"/></inertial>
+      <xacro:right_link_mesh visual_filename="package://openleg_description/meshes/right_leg/Right_Link6.stl" collision_filename="package://openleg_description/meshes/right_leg/Right_Link6.stl" xyz="0 0 0" rpy="0 0 ${pi}" scale="1 1 1" material="joint_dark"/>
+      <!-- Fusion inertia at COM, transformed into this URDF frame and scaled for the 0.95 kg total link mass. -->
+      <inertial><origin xyz="-0.004103 0.040339 0.077124"/><mass value="0.95"/><inertia ixx="0.000921950313" ixy="-0.000031496560" ixz="0.000005576139" iyy="0.000789173374" iyz="-0.000027795258" izz="0.000781461582"/></inertial>
     </link>
     <!-- J5: toes pitch, Link5 -> Link6 -->
     <joint name="right_joint5" type="revolute">
-      <parent link="right_link5"/><child link="right_link6"/><origin xyz="0 -0.054 0.18"/><axis xyz="0 1 0"/>
-      <limit lower="-${49 * pi / 360}" upper="${49 * pi / 360}" effort="140" velocity="10.47198"/>
+      <parent link="right_link5"/><child link="right_link6"/><origin xyz="0 -0.055 0.2"/><axis xyz="0 1 0"/>
+      <limit lower="-${49 * pi / 360}" upper="${49 * pi / 360}" effort="30" velocity="4.18879"/>
       <dynamics damping="2.0" friction="0.04"/>
     </joint>
@@ -88,25 +90,26 @@
       </visual>
       <collision>
-        <origin xyz="-0.01 0 0.055"/>
-        <geometry><box size="${foot_length} ${foot_collision_width} ${foot_height}"/></geometry>
+        <origin xyz="0 0 0" rpy="0 0 -${pi / 2}"/>
+        <geometry><mesh filename="package://openleg_description/meshes/right_leg/Link7.stl" scale="1 1 1"/></geometry>
       </collision>
+      <!-- Fusion inertia at COM, transformed into this URDF frame and scaled for the 0.50 kg total link mass. -->
       <inertial>
-        <origin xyz="0.025 0 -${foot_height / 2}"/><mass value="0.5"/>
-        <inertia ixx="${0.5 * (foot_width**2 + foot_height**2) / 12}" ixy="0" ixz="0" iyy="${0.5 * (foot_length**2 + foot_height**2) / 12}" iyz="0" izz="${0.5 * (foot_length**2 + foot_width**2) / 12}"/>
+        <origin xyz="-0.010 0 0.052"/><mass value="0.5"/>
+        <inertia ixx="0.000532780431" ixy="0" ixz="-0.000013684277" iyy="0.001459897118" iyz="0" izz="0.001621743391"/>
       </inertial>
     </link>
     <!-- J6: toes roll, Link6 -> Link7 -->
     <joint name="right_joint6" type="revolute">
-      <parent link="right_link6"/><child link="right_link7"/><origin xyz="0.03712500 0.0385 0.12097726"/><axis xyz="1 0 0"/>
-      <limit lower="-${pi / 6}" upper="${pi / 6}" effort="97" velocity="4.18879"/>
+      <parent link="right_link6"/><child link="right_link7"/><origin xyz="0.032 0.043 0.08"/><axis xyz="1 0 0"/>
+      <limit lower="-${pi / 6}" upper="${pi / 6}" effort="30" velocity="4.18879"/>
       <dynamics damping="2.0" friction="0.04"/>
     </joint>
-    <gazebo reference="right_link1"><mu1>2.5</mu1><mu2>2.5</mu2><kp>200000</kp><kd>1000</kd><maxVel>0.05</maxVel><minDepth>0.001</minDepth></gazebo>
-    <gazebo reference="right_link2"><mu1>2.5</mu1><mu2>2.5</mu2><kp>200000</kp><kd>1000</kd><maxVel>0.05</maxVel><minDepth>0.001</minDepth></gazebo>
-    <gazebo reference="right_link3"><mu1>2.5</mu1><mu2>2.5</mu2><kp>200000</kp><kd>1000</kd><maxVel>0.05</maxVel><minDepth>0.001</minDepth></gazebo>
-    <gazebo reference="right_link4"><mu1>2.5</mu1><mu2>2.5</mu2><kp>200000</kp><kd>1000</kd><maxVel>0.05</maxVel><minDepth>0.001</minDepth></gazebo>
-    <gazebo reference="right_link5"><mu1>2.5</mu1><mu2>2.5</mu2><kp>200000</kp><kd>1000</kd><maxVel>0.05</maxVel><minDepth>0.001</minDepth></gazebo>
-    <gazebo reference="right_link6"><mu1>2.5</mu1><mu2>2.5</mu2><kp>200000</kp><kd>1000</kd><maxVel>0.05</maxVel><minDepth>0.001</minDepth></gazebo>
-    <gazebo reference="right_link7"><mu1>1.2</mu1><mu2>1.2</mu2><kp>200000</kp><kd>1000</kd><maxVel>0.05</maxVel><minDepth>0.001</minDepth></gazebo>
+    <gazebo reference="right_link1"><mu1>0.5</mu1><mu2>0.5</mu2><kp>200000</kp><kd>1000</kd><maxVel>0.05</maxVel><minDepth>0.001</minDepth></gazebo>
+    <gazebo reference="right_link2"><mu1>0.5</mu1><mu2>0.5</mu2><kp>200000</kp><kd>1000</kd><maxVel>0.05</maxVel><minDepth>0.001</minDepth></gazebo>
+    <gazebo reference="right_link3"><mu1>0.5</mu1><mu2>0.5</mu2><kp>200000</kp><kd>1000</kd><maxVel>0.05</maxVel><minDepth>0.001</minDepth></gazebo>
+    <gazebo reference="right_link4"><mu1>0.5</mu1><mu2>0.5</mu2><kp>200000</kp><kd>1000</kd><maxVel>0.05</maxVel><minDepth>0.001</minDepth></gazebo>
+    <gazebo reference="right_link5"><mu1>0.5</mu1><mu2>0.5</mu2><kp>200000</kp><kd>1000</kd><maxVel>0.05</maxVel><minDepth>0.001</minDepth></gazebo>
+    <gazebo reference="right_link6"><mu1>0.5</mu1><mu2>0.5</mu2><kp>200000</kp><kd>1000</kd><maxVel>0.05</maxVel><minDepth>0.001</minDepth></gazebo>
+    <gazebo reference="right_link7"><mu1>0.9</mu1><mu2>0.9</mu2><kp>200000</kp><kd>1000</kd><maxVel>0.05</maxVel><minDepth>0.001</minDepth></gazebo>
   </xacro:macro>
 </robot>
