Commit message: Update robot CAD alignment, inertial properties, and contact settings
  - Mirror right-leg joint origins and mesh alignment onto the left leg
  - Update base and right-leg COMs and inertia tensors from CAD data
  - Add 500 g allowances to updated parts except Link 6
  - Mirror right-leg masses, COMs, and inertia tensors onto the left leg
  - Revise joint limits on both legs
  - Move the IMU to 180 mm above the base origin
  - Set provisional TPU foot friction to 0.8
  - Fix stale left-leg mesh references and update the IMU pose test

File: urdf/right_leg.urdf.xacro (robot description, xacro)
@@ -18,6 +18,15 @@
     <link name="right_link1">
       <xacro:right_link_mesh visual_filename="package://openleg_description/meshes/right_leg/Right_Link1.stl" collision_filename="package://openleg_description/meshes/right_leg/Right_Link1.stl" xyz="0 0 0" rpy="${pi / 2} 0 ${pi / 2}" scale="1 1 1" material="right_leg_red"/>
-      <!-- Fusion inertia at COM, transformed into this URDF frame and scaled for the 1.95 kg total link mass. -->
-      <inertial><origin xyz="0.035 0 0"/><mass value="1.95"/><inertia ixx="0.003758080176" ixy="0.000113110329" ixz="0.000018626355" iyy="0.002425144326" iyz="0.000082610274" izz="0.002891882116"/></inertial>
+      <!-- CAD mass: 1.674577 kg, plus 0.5 kg for bolts and wires.
+           CAD X/Y/Z map to URDF Y/Z/X; CAD and link origins coincide.
+           Inertia at COM is converted from g mm^2 to kg m^2, then scaled
+           assuming the added mass follows the CAD mass distribution; COM is unchanged. -->
+      <xacro:property name="right_link1_inertia_scale" value="${(1.674577 + 0.5) / 1.674577}"/>
+      <inertial>
+        <origin xyz="0.029177 -0.000018 -0.001849" rpy="0 0 0"/>
+        <mass value="${1.674577 + 0.5}"/>
+        <inertia ixx="${0.003013000000 * right_link1_inertia_scale}" ixy="${-0.000000570932 * right_link1_inertia_scale}" ixz="${-0.000074828761 * right_link1_inertia_scale}"
+                 iyy="${0.001887000000 * right_link1_inertia_scale}" iyz="${-0.000000030342 * right_link1_inertia_scale}" izz="${0.002170000000 * right_link1_inertia_scale}"/>
+      </inertial>
     </link>
     <joint name="right_base_fixed_joint" type="fixed">
@@ -27,5 +36,15 @@
     <link name="right_link2">
       <xacro:right_link_mesh visual_filename="package://openleg_description/meshes/right_leg/Right_Link2.stl" collision_filename="package://openleg_description/meshes/right_leg/Right_Link2.stl" xyz="0 0 0" rpy="0 0 0" scale="1 1 1" material="right_leg_red"/>
-      <inertial><origin xyz="0 0.068 0"/><mass value="1.75"/><inertia ixx="0.003134759430" ixy="-0.000015824529" ixz="-0.000001019248" iyy="0.001856093868" iyz="-0.000000151933" izz="0.002351329675"/></inertial>
+      <!-- CAD mass: 1.760088 kg, plus 0.5 kg for bolts and wires.
+           CAD X/Y/Z map to URDF X/Z/-Y; CAD and link origins coincide.
+           Inertia at COM is converted from g mm^2 to kg m^2, then scaled
+           assuming the added mass follows the CAD mass distribution; COM is unchanged. -->
+      <xacro:property name="right_link2_inertia_scale" value="${(1.760088 + 0.5) / 1.760088}"/>
+      <inertial>
+        <origin xyz="0.001703 0.056011 0.048374" rpy="0 0 0"/>
+        <mass value="${1.760088 + 0.5}"/>
+        <inertia ixx="${0.003362000000 * right_link2_inertia_scale}" ixy="${-0.000012697179 * right_link2_inertia_scale}" ixz="${-0.000018817964 * right_link2_inertia_scale}"
+                 iyy="${0.002249000000 * right_link2_inertia_scale}" iyz="${-0.000324300000 * right_link2_inertia_scale}" izz="${0.002256000000 * right_link2_inertia_scale}"/>
+      </inertial>
     </link>
     <!-- J1: hip pitch, Link1 -> Link2 -->
@@ -33,5 +52,5 @@
       <parent link="right_link1"/><child link="right_link2"/>
       <origin xyz="0.064 0 0" rpy="0 ${pi} -${pi / 2}"/><axis xyz="0 1 0"/>
-      <limit lower="-0.915" upper="${-0.915 + 5 * pi / 6}" effort="40" velocity="5.23599"/>
+      <limit lower="${-90 * pi / 180}" upper="${90 * pi / 180}" effort="40" velocity="5.23599"/>
       <dynamics damping="2.0" friction="0.05"/>
     </joint>
@@ -42,13 +61,20 @@
     <!-- J2: hip roll, Link2 -> Link3 -->
     <joint name="right_joint2" type="revolute">
-      <parent link="right_link2"/><child link="right_link3"/><origin xyz="-0.027 0.075 0" rpy="0 0 0"/><axis xyz="1 0 0"/>
-      <limit lower="-${pi / 2}" upper="${5 * pi / 36}" effort="40" velocity="5.23599"/>
+      <parent link="right_link2"/><child link="right_link3"/><origin xyz="-0.027 0.060 0.055" rpy="0 0 0"/><axis xyz="1 0 0"/>
+      <limit lower="${-60 * pi / 180}" upper="${30 * pi / 180}" effort="40" velocity="5.23599"/>
       <dynamics damping="2.0" friction="0.05"/>
     </joint>
     <link name="right_link4">
       <xacro:right_link_mesh visual_filename="package://openleg_description/meshes/right_leg/Right_Link4.stl" collision_filename="package://openleg_description/meshes/right_leg/Right_Link4.stl" xyz="0 0 0" rpy="-${pi / 2} 0 -${pi / 2}" scale="1 1 1" material="right_leg_red"/>
+      <!-- CAD mass: 2.826622 kg, plus 0.5 kg for bolts and wires.
+           CAD X/Y/Z map to URDF -Y/X/Z; CAD and link origins coincide.
+           Inertia at COM is converted from g mm^2 to kg m^2, then scaled
+           assuming the added mass follows the CAD mass distribution; COM is unchanged. -->
+      <xacro:property name="right_link4_inertia_scale" value="${(2.826622 + 0.5) / 2.826622}"/>
       <inertial>
-        <origin xyz="0 -0.015 0.109"/><mass value="3.0"/>
-        <inertia ixx="0.011445270031" ixy="-0.000000623481" ixz="-0.000025390890" iyy="0.012149594340" iyz="0.001008737419" izz="0.003608626316"/>
+        <origin xyz="-0.000012 -0.015481 0.108918" rpy="0 0 0"/>
+        <mass value="${2.826622 + 0.5}"/>
+        <inertia ixx="${0.010770000000 * right_link4_inertia_scale}" ixy="${-0.000000610697 * right_link4_inertia_scale}" ixz="${-0.000024502364 * right_link4_inertia_scale}"
+                 iyy="${0.011520000000 * right_link4_inertia_scale}" iyz="${0.000848900000 * right_link4_inertia_scale}" izz="${0.003316000000 * right_link4_inertia_scale}"/>
       </inertial>
     </link>
@@ -60,8 +86,15 @@
     </joint>
     <link name="right_link5">
-      <xacro:right_link_mesh visual_filename="package://openleg_description/meshes/right_leg/Link5.stl" collision_filename="package://openleg_description/meshes/right_leg/Link5.stl" xyz="0 0 0" rpy="0 -${pi / 2} 0" scale="1 1 1" material="right_leg_red"/>
+      <xacro:right_link_mesh visual_filename="package://openleg_description/meshes/right_leg/Right_Link5.stl" collision_filename="package://openleg_description/meshes/right_leg/Right_Link5.stl" xyz="0 0 0" rpy="0 -${pi / 2} 0" scale="1 1 1" material="right_leg_red"/>
+      <!-- CAD mass: 2.580937 kg, plus 0.5 kg for bolts and wires.
+           CAD X/Y/Z map to URDF Z/X/Y; CAD and link origins coincide.
+           Inertia at COM is converted from g mm^2 to kg m^2, then scaled
+           assuming the added mass follows the CAD mass distribution; COM is unchanged. -->
+      <xacro:property name="right_link5_inertia_scale" value="${(2.580937 + 0.5) / 2.580937}"/>
       <inertial>
-        <origin xyz="0 -0.014 0.129"/><mass value="1.94"/>
-        <inertia ixx="0.014234679170" ixy="-0.000000064992" ixz="-0.000000364381" iyy="0.013200580905" iyz="-0.000299782976" izz="0.002755133233"/>
+        <origin xyz="0.003961 -0.025956 0.151636" rpy="0 0 0"/>
+        <mass value="${2.580937 + 0.5}"/>
+        <inertia ixx="${0.014890000000 * right_link5_inertia_scale}" ixy="${0.000007623647 * right_link5_inertia_scale}" ixz="${-0.000082304091 * right_link5_inertia_scale}"
+                 iyy="${0.014170000000 * right_link5_inertia_scale}" iyz="${0.000764900000 * right_link5_inertia_scale}" izz="${0.002350000000 * right_link5_inertia_scale}"/>
       </inertial>
     </link>
@@ -69,16 +102,23 @@
     <joint name="right_joint4" type="revolute">
       <parent link="right_link4"/><child link="right_link5"/><origin xyz="0 0.012 0.147"/><axis xyz="0 1 0"/>
-      <limit lower="-${37 * pi / 72}" upper="${pi / 72}" effort="40" velocity="5.23599"/>
+      <limit lower="${-90 * pi / 180}" upper="${2 * pi / 180}" effort="40" velocity="5.23599"/>
       <dynamics damping="2.5" friction="0.05"/>
     </joint>
     <link name="right_link6">
       <xacro:right_link_mesh visual_filename="package://openleg_description/meshes/right_leg/Right_Link6.stl" collision_filename="package://openleg_description/meshes/right_leg/Right_Link6.stl" xyz="0 0 0" rpy="0 0 ${pi}" scale="1 1 1" material="joint_dark"/>
-      <!-- Fusion inertia at COM, transformed into this URDF frame and scaled for the 0.95 kg total link mass. -->
-      <inertial><origin xyz="-0.004103 0.040339 0.077124"/><mass value="0.95"/><inertia ixx="0.000921950313" ixy="-0.000031496560" ixz="0.000005576139" iyy="0.000789173374" iyz="-0.000027795258" izz="0.000781461582"/></inertial>
+      <!-- CAD mass: 0.079708 kg; Link6 has no added bolts/wires allowance.
+           CAD X/Y/Z map to URDF X/-Z/Y; CAD and link origins coincide.
+           Inertia at COM is converted from g mm^2 to kg m^2 without mass scaling. -->
+      <inertial>
+        <origin xyz="0 0.0185 -1.366e-13" rpy="0 0 0"/>
+        <mass value="0.079708"/>
+        <inertia ixx="0.000009707245" ixy="6.107e-16" ixz="7.369e-17"
+                 iyy="0.000006538190" iyz="0" izz="0.000014154792"/>
+      </inertial>
     </link>
     <!-- J5: toes pitch, Link5 -> Link6 -->
     <joint name="right_joint5" type="revolute">
-      <parent link="right_link5"/><child link="right_link6"/><origin xyz="0 -0.055 0.2"/><axis xyz="0 1 0"/>
-      <limit lower="-${49 * pi / 360}" upper="${49 * pi / 360}" effort="30" velocity="4.18879"/>
+      <parent link="right_link5"/><child link="right_link6"/><origin xyz="0 -0.0475 0.27"/><axis xyz="0 1 0"/>
+      <limit lower="${-25 * pi / 180}" upper="${20 * pi / 180}" effort="30" velocity="4.18879"/>
       <dynamics damping="2.0" friction="0.04"/>
     </joint>
@@ -93,14 +133,20 @@
         <geometry><mesh filename="package://openleg_description/meshes/right_leg/Link7.stl" scale="1 1 1"/></geometry>
       </collision>
-      <!-- Fusion inertia at COM, transformed into this URDF frame and scaled for the 0.50 kg total link mass. -->
+      <!-- CAD mass: 0.714171 kg, plus 0.5 kg for bolts and wires.
+           CAD X/Y/Z map to URDF -Y/-Z/X; CAD and link origins coincide.
+           Inertia at COM is converted from g mm^2 to kg m^2, then scaled
+           assuming the added mass follows the CAD mass distribution; COM is unchanged. -->
+      <xacro:property name="right_link7_inertia_scale" value="${(0.714171 + 0.5) / 0.714171}"/>
       <inertial>
-        <origin xyz="-0.010 0 0.052"/><mass value="0.5"/>
-        <inertia ixx="0.000532780431" ixy="0" ixz="-0.000013684277" iyy="0.001459897118" iyz="0" izz="0.001621743391"/>
+        <origin xyz="-0.019854 0 0.021463" rpy="0 0 0"/>
+        <mass value="${0.714171 + 0.5}"/>
+        <inertia ixx="${0.000589000000 * right_link7_inertia_scale}" ixy="${-0.000000072115 * right_link7_inertia_scale}" ixz="${-0.000112700000 * right_link7_inertia_scale}"
+                 iyy="${0.001700000000 * right_link7_inertia_scale}" iyz="${0.000000004097 * right_link7_inertia_scale}" izz="${0.002004000000 * right_link7_inertia_scale}"/>
       </inertial>
     </link>
     <!-- J6: toes roll, Link6 -> Link7 -->
     <joint name="right_joint6" type="revolute">
-      <parent link="right_link6"/><child link="right_link7"/><origin xyz="0.032 0.043 0.08"/><axis xyz="1 0 0"/>
-      <limit lower="-${pi / 6}" upper="${pi / 6}" effort="30" velocity="4.18879"/>
+      <parent link="right_link6"/><child link="right_link7"/><origin xyz="0.015 0.0185 0.00"/><axis xyz="1 0 0"/>
+      <limit lower="${-15 * pi / 180}" upper="${15 * pi / 180}" effort="30" velocity="4.18879"/>
       <dynamics damping="2.0" friction="0.04"/>
     </joint>
@@ -111,5 +157,6 @@
     <gazebo reference="right_link5"><mu1>0.5</mu1><mu2>0.5</mu2><kp>200000</kp><kd>1000</kd><maxVel>0.05</maxVel><minDepth>0.001</minDepth></gazebo>
     <gazebo reference="right_link6"><mu1>0.5</mu1><mu2>0.5</mu2><kp>200000</kp><kd>1000</kd><maxVel>0.05</maxVel><minDepth>0.001</minDepth></gazebo>
-    <gazebo reference="right_link7"><mu1>0.9</mu1><mu2>0.9</mu2><kp>200000</kp><kd>1000</kd><maxVel>0.05</maxVel><minDepth>0.001</minDepth></gazebo>
+    <!-- TPU sole: both tangential friction directions use the shared foot_friction estimate. -->
+    <gazebo reference="right_link7"><mu1>${foot_friction}</mu1><mu2>${foot_friction}</mu2><kp>200000</kp><kd>1000</kd><maxVel>0.05</maxVel><minDepth>0.001</minDepth></gazebo>
   </xacro:macro>
 </robot>
