Commit message: fix(sim): remove stale waist and torso controller joints

File: urdf/main.urdf.xacro (robot description, xacro)
@@ -5,8 +5,4 @@
   <!-- Change these dimensions first when adapting the model to the real hardware. -->
   <xacro:property name="base_mass" value="${4.264361 + 0.5}"/>
-  <!-- EDITABLE: replace with the measured upper-body inertial data. -->
-  <xacro:property name="upper_body_mass" value="3.4"/>
-  <!-- EDITABLE: replace with the measured torso inertial data. -->
-  <xacro:property name="torso_mass" value="5.5"/>
   <xacro:property name="pelvis_x" value="0.18"/>
   <xacro:property name="pelvis_y" value="0.23358873"/>
@@ -88,6 +84,4 @@
       <xacro:position_controlled_joint joint_name="right_joint5"/>
       <xacro:position_controlled_joint joint_name="right_joint6"/>
-      <xacro:position_controlled_joint joint_name="waist_joint"/>
-      <xacro:position_controlled_joint joint_name="torso_pitch_joint"/>
     </ros2_control>
     <!-- Simulated body IMU, mounted 180 mm above the base-link origin. -->
@@ -103,12 +97,4 @@
       </sensor>
     </gazebo>
-    <gazebo reference="upper_body_link">
-      <mu1>0.5</mu1><mu2>0.5</mu2>
-      <kp>200000</kp><kd>1000</kd><maxVel>0.05</maxVel><minDepth>0.001</minDepth>
-    </gazebo>
-    <gazebo reference="torso_link">
-      <mu1>0.5</mu1><mu2>0.5</mu2>
-      <kp>200000</kp><kd>1000</kd><maxVel>0.05</maxVel><minDepth>0.001</minDepth>
-    </gazebo>
     <gazebo>
       <plugin filename="libgz_ros2_control-system.so" name="gz_ros2_control::GazeboSimROS2ControlPlugin">
